Commit message: problem solving left

File: src/hola_bot/urdf/hola_bot.urdf (robot description, URDF)
Before this commit: robot hola_bot, 2 links, 0 joints
Joints:
- added joint front_joint: type continuous, parent base_link, child front_wheel, origin xyz=0 0.17483 -0.0335 rpy=0 0 0, axis 0 -1 0, limit effort=5 velocity=5

Commit message: wheel joints determined

File: src/hola_bot/urdf/hola_bot.urdf (robot description, URDF)
Before this commit: robot hola_bot, 2 links, 1 joints
Links:
- added link left_wheel, mass 0.062; collision cylinder length=0.02 radius=.03; visual mesh filename=package://hola_bot/meshes/wheel.STL
- added link right_wheel, mass 0.062; collision cylinder length=0.02 radius=.03; visual mesh filename=package://hola_bot/meshes/wheel.STL
- link base_link: geometry collision cylinder length=0.005 radius=0.15; visual mesh filename=package://hola_bot/meshes/base_link.STL
Joints:
- added joint left_joint: type continuous, parent base_link, child left_wheel, origin xyz=-0.15154 -0.087275 -0.0335 rpy=0 0 0, axis 0 -1 0, limit effort=5 velocity=5
- added joint right_joint: type continuous, parent base_link, child right_wheel, origin xyz=0.15154 -0.087275 -0.0335 rpy=0 0 0, axis 0 -1 0, limit effort=5 velocity=5

Commit message: right whell perfectly done

File: src/hola_bot/urdf/hola_bot.urdf (robot description, URDF)
Before this commit: robot hola_bot, 4 links, 3 joints
Joints:
- joint left_joint: origin xyz=-0.15154 -0.087275 -0.0335 rpy=0 0 0 -> xyz=-0.15154 -0.087275 -0.0335 rpy=0 0 1
- joint right_joint: origin xyz=0.15154 -0.087275 -0.0335 rpy=0 0 0 -> xyz=0.14054 -0.082275 -0.0335 rpy=0 0 1

Commit message: gzebo part perfectly done

File: src/hola_bot/urdf/hola_bot.urdf (robot description, URDF)
Before this commit: robot hola_bot, 4 links, 3 joints
Joints:
- joint left_joint: origin xyz=-0.15154 -0.087275 -0.0335 rpy=0 0 1 -> xyz=-0.14054 -0.082275 -0.0335 rpy=0 0 -1
